Commit message: feat: Add Autonomous Drive

File: robot/src/my_cartographer/urdf/my_robot.urdf (robot description, URDF)
Before this commit: robot my_robot, 3 links, 2 joints
Links:
- added link front_marker; visual box size=0.08 0.02 0.02
- link base_link: mass None -> 5.0; geometry collision box size=0.40 0.30 0.28; visual box size=0.40 0.30 0.28
- link imu_link: geometry collision box size=0.02 0.02 0.01; visual box size=0.02 0.02 0.01
- link laser_frame: geometry collision cylinder length=0.05 radius=0.03; visual cylinder length=0.05 radius=0.03
Joints:
- added joint base_link_to_front_marker: type fixed, parent base_link, child front_marker, origin xyz=0.22 0.0 0.14 rpy=0 0 0
- joint base_link_to_imu_link: origin xyz=0.0 0.0 0.0 rpy=0 0 0 -> xyz=0 0 0 rpy=0 0 0
- joint base_link_to_laser_frame: origin xyz=0.0 0.0 0.1 rpy=0 0 0 -> xyz=0.05 0.0 0.28 rpy=0 0 0
